File: ToF_camera_VGA.sch (KiCad schematic (older format))
At the start: 51 parts, among them J1 Conn_01x22, J2 Conn_01x08, J8 Conn_01x02, SW1 SW_Push, U1 TPS82150, U2 MLX75027, U3 TPS82150, U4 TPS82150, U5 TPSM84624, U6 PCA9306, Y1 Crystal

Commit message: Inverted connector and re-routed CSI-2 lanes
Connections:
- wire segments 485 -> 453
- no-connect marks 5 -> 6
Other:
- note added: "+3.3v -1\nSDA - 2\nSCL - 3"
- note added: "15 - +3.3 V\n14 - SDA \n13 - SCL\n12 - GPIO1\n11 - GPIO0\n10 - GND\n9 - CLK+\n8 - CLK-\n7 - GND\n6 - D1+\n5 - D1-\n4 - GND\n3 - D0+\n2 - D0-\n1 - GND"
- note added: "GND - 13\nCLK+ - 14\nCLK- - 15\nGND - 16\nD1+ - 17\nD1- - 18\nGND - 19\nD0+ - 20\nD0- - 21\nGND - 22"
- note added: "GND - 7\nD3+ - 8\nD3- - 9\nGND - 10\nD2+ - 11\nD2- - 12"
- note added: "GPIO1 -5\nGPIO0 -6"
- note added: "It isn't exact drawing, but connectors should be connected in similar way using standard Raspberry Pi cable-adapter"
- note added: "J3 connector on Zynqberry is rotated, so that our connector can be drawn in regular manner"
- note added: "nc - 4"
- moved on the sheet: J1, J8

Commit message: Almost there... minor modifications for production needed
Parts:
- removed J2: Conn_01x08, Pin_Headers:Pin_Header_Straight_1x08_Pitch2.54mm, symbol Connector_Generic:Conn_01x08
- added J2, J4: Conn_01x01, Pin_Headers:Pin_Header_Straight_1x01_Pitch2.54mm, symbol Connector_Generic:Conn_01x01
- added J3, J5, J6: Conn_01x04, Pin_Headers:Pin_Header_Straight_1x04_Pitch2.54mm, symbol Connector_Generic:Conn_01x04
- added R17: R, Resistors_SMD:R_0805, symbol Device:R
- J8: footprint Pin_Headers:Pin_Header_Straight_1x02_Pitch2.54mm -> Resistors_SMD:R_0201_NoSilk
Connections:
- net labels added: PGOOD_1.8V, PGOOD_VDDA
- wire segments 453 -> 473
Changed lines of the file:
@@
 Wire Wire Line
 	4000 6650 4350 6650
-$Comp
-L Connector_Generic:Conn_01x08 J2
-U 1 1 5D7435B4
-P 2650 7150
-F 0 "J2" H 2568 6525 50  0000 C CNN
-F 1 "Conn_01x08" H 2568 6616 50  0000 C CNN
-F 2 "Pin_Headers:Pin_Header_Straight_1x08_Pitch2.54mm" H 2650 7150 50  0001 C CNN
-F 3 "~" H 2650 7150 50  0001 C CNN
-	1    2650 7150
-	-1   0    0    1
-$EndComp
 Wire Wire Line
 	2850 6750 4350 6750
 Connection ~ 3350 6850
-Wire Wire Line
-	2850 6950 3050 6950
 Connection ~ 3050 6950
 Wire Wire Line
@@
 Wire Wire Line
 	4350 7250 2850 7250
-Wire Wire Line
-	2850 7450 4350 7450
 Wire Wire Line
 	4100 7550 4200 7550
@@
 	4200 7550 4200 7800
 Wire Wire Line
-	4200 7800 3050 7800
-Wire Wire Line
-	3050 7800 3050 7350
-Wire Wire Line
-	3050 7350 2850 7350
+	4200 7800 3400 7800
 Connection ~ 4200 7550
 Wire Wire Line
@@
 Connection ~ 12100 4400
 Text Label 12250 5100 0    50   ~ 0
-PGOOD_VDD
+PGOOD_1.8V
 Wire Wire Line
 	12250 5100 11750 5100
@@
 Connection ~ 3850 4450
 Text Label 4000 5150 0    50   ~ 0
-PGOOD_VDD
+PGOOD_VDDA
 Wire Wire Line
 	4000 5150 3500 5150
@@
 F 0 "J8" H 6580 1542 50  0000 L CNN
 F 1 "Conn_01x02" H 6580 1451 50  0000 L CNN
-F 2 "Pin_Headers:Pin_Header_Straight_1x02_Pitch2.54mm" H 6500 1550 50  0001 C CNN
+F 2 "Resistors_SMD:R_0201_NoSilk" H 6500 1550 50  0001 C CNN
 F 3 "~" H 6500 1550 50  0001 C CNN
 	1    6500 1550
@@
 Wire Wire Line
 	2850 5300 3850 5300
-Wire Wire Line
-	2300 6850 2850 6850
-Connection ~ 2850 6850
-Wire Wire Line
-	2850 6850 3350 6850
-Wire Wire Line
-	2300 6950 2850 6950
-Connection ~ 2850 6950
 Wire Wire Line
 	3050 6250 3050 6350
@@
 	2350 6750 2300 6750
 Wire Wire Line
-	3050 6250 2900 6250
+	3050 6250 2950 6250
 Wire Wire Line
 	2600 6250 2350 6250
@@
 It isn't exact drawing, but connectors should be connected in similar way using standard Raspberry Pi cable-adapter
 $Comp
-L power:GNDD #PWR?
+L power:GNDD #PWR0122
 U 1 1 5D9DAA50
 P 1900 7350
-F 0 "#PWR?" H 1900 7100 50  0001 C CNN
+F 0 "#PWR0122" H 1900 7100 50  0001 C CNN
 F 1 "GNDD" H 1904 7195 50  0000 C CNN
 F 2 "" H 1900 7350 50  0001 C CNN
@@
 Wire Wire Line
 	6650 1950 6650 2250
+$Comp
+L Connector_Generic:Conn_01x04 J3
+U 1 1 5DF82595
+P 2650 7250
+F 0 "J3" H 2568 6825 50  0000 C CNN
+F 1 "Conn_01x04" H 2568 6916 50  0000 C CNN
+F 2 "Pin_Headers:Pin_Header_Straight_1x04_Pitch2.54mm" H 2650 7250 50  0001 C CNN
+F 3 "~" H 2650 7250 50  0001 C CNN
+	1    2650 7250
+	-1   0    0    1
+$EndComp
+Wire Wire Line
+	2300 6950 3050 6950
+Wire Wire Line
+	2300 6850 3350 6850
+Wire Wire Line
+	4350 7450 3100 7450
+Wire Wire Line
+	3100 7450 3100 7350
+Wire Wire Line
+	3100 7350 2850 7350
+$Comp
+L Device:R R17
+U 1 1 5E0FFBBD
+P 3200 7600
+F 0 "R17" V 2993 7600 50  0000 C CNN
+F 1 "R" V 3084 7600 50  0000 C CNN
+F 2 "Resistors_SMD:R_0805" V 3130 7600 50  0001 C CNN
+F 3 "~" H 3200 7600 50  0001 C CNN
+	1    3200 7600
+	0    1    1    0
+$EndComp
+Wire Wire Line
+	2950 6250 2950 7600
+Wire Wire Line
+	2950 7600 3050 7600
+Connection ~ 2950 6250
+Wire Wire Line
+	2950 6250 2900 6250
+Wire Wire Line
+	3350 7600 3400 7600
+Wire Wire Line
+	3400 7600 3400 7800
+Connection ~ 3400 7800
+Wire Wire Line
+	3400 7800 3050 7800
+$Comp
+L Connector_Generic:Conn_01x01 J4
+U 1 1 5E1730FD
+P 2850 7800
+F 0 "J4" H 2768 7575 50  0000 C CNN
+F 1 "Conn_01x01" H 2768 7666 50  0000 C CNN
+F 2 "Pin_Headers:Pin_Header_Straight_1x01_Pitch2.54mm" H 2850 7800 50  0001 C CNN
+F 3 "~" H 2850 7800 50  0001 C CNN
+	1    2850 7800
+	-1   0    0    1
+$EndComp
+$Comp
+L Connector_Generic:Conn_01x01 J2
+U 1 1 5E1738BE
+P 2650 6750
+F 0 "J2" H 2568 6525 50  0000 C CNN
+F 1 "Conn_01x01" H 2568 6616 50  0000 C CNN
+F 2 "Pin_Headers:Pin_Header_Straight_1x01_Pitch2.54mm" H 2650 6750 50  0001 C CNN
+F 3 "~" H 2650 6750 50  0001 C CNN
+	1    2650 6750
+	-1   0    0    1
+$EndComp
+$Comp
+L Connector_Generic:Conn_01x04 J5
+U 1 1 5E1916FE
+P 9200 1650
+F 0 "J5" H 9118 1225 50  0000 C CNN
+F 1 "Conn_01x04" H 9118 1316 50  0000 C CNN
+F 2 "Pin_Headers:Pin_Header_Straight_1x04_Pitch2.54mm" H 9200 1650 50  0001 C CNN
+F 3 "~" H 9200 1650 50  0001 C CNN
+	1    9200 1650
+	-1   0    0    1
+$EndComp
+$Comp
+L Connector_Generic:Conn_01x04 J6
+U 1 1 5E1961FC
+P 9200 2500
+F 0 "J6" H 9118 2075 50  0000 C CNN
+F 1 "Conn_01x04" H 9118 2166 50  0000 C CNN
+F 2 "Pin_Headers:Pin_Header_Straight_1x04_Pitch2.54mm" H 9200 2500 50  0001 C CNN
+F 3 "~" H 9200 2500 50  0001 C CNN
+	1    9200 2500
+	-1   0    0    1
+$EndComp
+$Comp
+L power:+12V #PWR0123
+U 1 1 5E196C75
+P 9550 1350
+F 0 "#PWR0123" H 9550 1200 50  0001 C CNN
+F 1 "+12V" H 9565 1523 50  0000 C CNN
+F 2 "" H 9550 1350 50  0001 C CNN
+F 3 "" H 9550 1350 50  0001 C CNN
+	1    9550 1350
+	1    0    0    -1
+$EndComp
+$Comp
+L power:GNDD #PWR0124
+U 1 1 5E1971BC
+P 9550 2700
+F 0 "#PWR0124" H 9550 2450 50  0001 C CNN
+F 1 "GNDD" H 9554 2545 50  0000 C CNN
+F 2 "" H 9550 2700 50  0001 C CNN
+F 3 "" H 9550 2700 50  0001 C CNN
+	1    9550 2700
+	1    0    0    -1
+$EndComp
+Wire Wire Line
+	9400 1450 9550 1450
+Wire Wire Line
+	9550 1450 9550 1350
+Wire Wire Line
+	9400 1750 9550 1750
+Connection ~ 9550 1450
+Wire Wire Line
+	9400 1550 9550 1550
+Connection ~ 9550 1550
+Wire Wire Line
+	9550 1550 9550 1450
+Wire Wire Line
+	9400 1650 9550 1650
+Wire Wire Line
+	9550 1550 9550 1650
+Connection ~ 9550 1650
+Wire Wire Line
+	9550 1650 9550 1750
+Wire Wire Line
+	9400 2300 9550 2300
+Wire Wire Line
+	9550 2300 9550 2400
+Wire Wire Line
+	9400 2400 9550 2400
+Connection ~ 9550 2400
+Wire Wire Line
+	9550 2400 9550 2500
+Wire Wire Line
+	9400 2500 9550 2500
+Connection ~ 9550 2500
+Wire Wire Line
+	9550 2500 9550 2600
+Wire Wire Line
+	9400 2600 9550 2600
+Connection ~ 9550 2600
+Wire Wire Line
+	9550 2600 9550 2700
 $EndSCHEMATC

Commit message: Added filter between analog and digital grounds. Moved to 5.1.4 KiCad version
Parts:
- added L1: L, Inductors:Inductor_1212, symbol Device:L
Connections:
- net GNDA: now also L1.1
- net GNDD: now also L1.2
Changed lines of the file:
@@
 EESchema Schematic File Version 4
 LIBS:ToF_camera_VGA-cache
-EELAYER 29 0
+EELAYER 30 0
 EELAYER END
 $Descr A3 16535 11693
@@
 Wire Wire Line
 	9550 2600 9550 2700
+$Comp
+L Device:L L1
+U 1 1 5D5EC021
+P 4850 5300
+F 0 "L1" V 5040 5300 50  0000 C CNN
+F 1 "L" V 4949 5300 50  0000 C CNN
+F 2 "Inductors:Inductor_1212" H 4850 5300 50  0001 C CNN
+F 3 "~" H 4850 5300 50  0001 C CNN
+	1    4850 5300
+	0    -1   -1   0
+$EndComp
+Wire Wire Line
+	5000 5300 5800 5300
+Connection ~ 5800 5300
+Wire Wire Line
+	4700 5300 3850 5300
+Connection ~ 3850 5300
 $EndSCHEMATC

Commit message: Updated BOM
Parts:
- C10, C14, C3: value 3.3n -> 430p, 1m
- C16: footprint Capacitors_SMD:CP_Elec_4x5.8 -> Capacitors_SMD:CP_Elec_5x5.8
- C9: value 10u -> 10u, 2.229 mOhm
- R1, R17, R2: value R -> 10k
- R4: value 124k -> 237k
- R7: value 124k -> 49.9k
- Y1: footprint Crystals:Crystal_SMD_2012-2pin_2.0x1.2mm -> Crystals:Crystal_SMD_5032-2pin_5.0x3.2mm
Other:
- note added: "C3, C10 and C14\n 430pF or 3.3nF???\n"
- note removed: "BAD COMPONENT VALUES!!!\n"
Changed lines of the file:
@@
 P 3350 6550
 F 0 "R2" H 3420 6596 50  0000 L CNN
-F 1 "R" H 3420 6505 50  0000 L CNN
+F 1 "10k" H 3420 6505 50  0000 L CNN
 F 2 "Resistors_SMD:R_0805" V 3280 6550 50  0001 C CNN
 F 3 "~" H 3350 6550 50  0001 C CNN
@@
 P 3050 6550
 F 0 "R1" H 3120 6596 50  0000 L CNN
-F 1 "R" H 3120 6505 50  0000 L CNN
+F 1 "10k" H 3120 6505 50  0000 L CNN
 F 2 "Resistors_SMD:R_0805" V 2980 6550 50  0001 C CNN
 F 3 "~" H 3050 6550 50  0001 C CNN
@@
 F 0 "Y1" H 3850 7618 50  0000 C CNN
 F 1 "Crystal" H 3850 7527 50  0000 C CNN
-F 2 "Crystals:Crystal_SMD_2012-2pin_2.0x1.2mm" H 3850 7350 50  0001 C CNN
+F 2 "Crystals:Crystal_SMD_5032-2pin_5.0x3.2mm" H 3850 7350 50  0001 C CNN
 F 3 "~" H 3850 7350 50  0001 C CNN
 	1    3850 7350
@@
 P 5800 4650
 F 0 "C9" H 5915 4696 50  0000 L CNN
-F 1 "10u" H 5915 4605 50  0000 L CNN
+F 1 "10u, 2.229 mOhm" H 5915 4605 50  0000 L CNN
 F 2 "Capacitors_SMD:C_0805" H 5838 4500 50  0001 C CNN
 F 3 "~" H 5800 4650 50  0001 C CNN
@@
 P 6050 5050
 F 0 "C10" H 6165 5096 50  0000 L CNN
-F 1 "3.3n" H 6165 5005 50  0000 L CNN
+F 1 "430p, 1m" H 6165 5005 50  0000 L CNN
 F 2 "Capacitors_SMD:C_0805" H 6088 4900 50  0001 C CNN
 F 3 "~" H 6050 5050 50  0001 C CNN
@@
 P 7250 4650
 F 0 "R7" V 7457 4650 50  0000 C CNN
-F 1 "124k" V 7366 4650 50  0000 C CNN
+F 1 "49.9k" V 7366 4650 50  0000 C CNN
 F 2 "Resistors_SMD:R_0805" V 7180 4650 50  0001 C CNN
 F 3 "~" H 7250 4650 50  0001 C CNN
@@
 P 10150 5000
 F 0 "C14" H 10265 5046 50  0000 L CNN
-F 1 "3.3n" H 10265 4955 50  0000 L CNN
+F 1 "430p, 1m" H 10265 4955 50  0000 L CNN
 F 2 "Capacitors_SMD:C_0805" H 10188 4850 50  0001 C CNN
 F 3 "~" H 10150 5000 50  0001 C CNN
@@
 $EndComp
 Text Notes 5150 3950 0    197  ~ 0
-BAD COMPONENT VALUES!!!\n
+C3, C10 and C14\n 430pF or 3.3nF???\n
 $Comp
 L Regulator_Switching:TPS82150 U1
@@
 P 1900 5050
 F 0 "C3" H 2015 5096 50  0000 L CNN
-F 1 "3.3n" H 2015 5005 50  0000 L CNN
+F 1 "430p, 1m" H 2015 5005 50  0000 L CNN
 F 2 "Capacitors_SMD:C_0805" H 1938 4900 50  0001 C CNN
 F 3 "~" H 1900 5050 50  0001 C CNN
@@
 P 3100 4650
 F 0 "R4" V 3307 4650 50  0000 C CNN
-F 1 "124k" V 3216 4650 50  0000 C CNN
+F 1 "237k" V 3216 4650 50  0000 C CNN
 F 2 "Resistors_SMD:R_0805" V 3030 4650 50  0001 C CNN
 F 3 "~" H 3100 4650 50  0001 C CNN
@@
 	4000 5150 3500 5150
 Connection ~ 3500 5150
-Text Notes 1000 3950 0    197  ~ 0
-BAD COMPONENT VALUES!!!\n
 $Comp
 L power:VDDA #PWR0117
@@
 F 0 "C16" H 11968 7946 50  0000 L CNN
 F 1 "220u" H 11968 7855 50  0000 L CNN
-F 2 "Capacitors_SMD:CP_Elec_4x5.8" H 11888 7750 50  0001 C CNN
+F 2 "Capacitors_SMD:CP_Elec_5x5.8" H 11888 7750 50  0001 C CNN
 F 3 "~" H 11850 7900 50  0001 C CNN
 	1    11850 7900
@@
 P 3200 7600
 F 0 "R17" V 2993 7600 50  0000 C CNN
-F 1 "R" V 3084 7600 50  0000 C CNN
+F 1 "10k" V 3084 7600 50  0000 C CNN
 F 2 "Resistors_SMD:R_0805" V 3130 7600 50  0001 C CNN
 F 3 "~" H 3200 7600 50  0001 C CNN

Commit message: Minor updates, production read. Added Gerbers
Parts:
- added R18: R, Resistors_SMD:R_0805, symbol Device:R
Connections:
- net VDDA: now also R18.1; no longer R4.2
- new net: R18.2, R4.2
Changed lines of the file:
@@
 Wire Wire Line
 	3500 4450 3500 4500
-Wire Wire Line
-	3250 4650 3350 4650
-Wire Wire Line
-	3350 4650 3350 4450
 Connection ~ 3350 4450
 Wire Wire Line
@@
 	4700 5300 3850 5300
 Connection ~ 3850 5300
+$Comp
+L Device:R R18
+U 1 1 5D64C9EF
+P 3350 4850
+F 0 "R18" H 3420 4896 50  0000 L CNN
+F 1 "R" H 3420 4805 50  0000 L CNN
+F 2 "Resistors_SMD:R_0805" V 3280 4850 50  0001 C CNN
+F 3 "~" H 3350 4850 50  0001 C CNN
+	1    3350 4850
+	1    0    0    -1
+$EndComp
+Wire Wire Line
+	3250 4650 3250 5000
+Wire Wire Line
+	3250 5000 3350 5000
+Wire Wire Line
+	3350 4450 3350 4700
 $EndSCHEMATC

Commit message: Version 2 with fixed following issues: 1. clock source added 2. Flat cable connector should be ok 3. I2C level shifter should be ok 4. Power tree simplified, 12 V needed only for VDDMIX, others are generated from 3.3 V on flat cable
Parts:
- removed C16: 220u, Capacitors_SMD:CP_Elec_5x5.8, symbol Device:CP
- removed J1: Conn_01x22, myFootprints:FPC_22, symbol Connector_Generic:Conn_01x22
- removed J8: Conn_01x02, Resistors_SMD:R_0201_NoSilk, symbol Connector_Generic:Conn_01x02
- removed JP1: SolderJumper_3_Open, Pin_Headers:Pin_Header_Straight_1x03_Pitch1.00mm_SMD_Pin1Right, symbol Jumper:SolderJumper_3_Open
- removed R10, R11: 10k, Resistors_SMD:R_0805, symbol Device:R
- removed R12: 124k, Resistors_SMD:R_0805, symbol Device:R
- removed R13, R5, R8: 100k, Resistors_SMD:R_0402, symbol Device:R
- removed R14: 4.12k, Resistors_SMD:R_0805, symbol Device:R
- removed R15: 110k, Resistors_SMD:R_0805, symbol Device:R
- removed R16: 200k, Resistors_SMD:R_0805, symbol Device:R
- removed R18: R, Resistors_SMD:R_0805, symbol Device:R
- removed R4: 237k, Resistors_SMD:R_0805, symbol Device:R
- removed R9: 100k, Resistors_SMD:R_0805, symbol Device:R
- removed U1, U3, U4: TPS82150, myFootprints:TPS82130, symbol Regulator_Switching:TPS82150
- removed U5: TPSM84624, myFootprints:TPSM84624, symbol myParts:TPSM84624
- removed U6: PCA9306, Housings_SSOP:SSOP-8_2.95x2.8mm_Pitch0.65mm, symbol Interface:PCA9306
- removed Y1: Crystal, Crystals:Crystal_SMD_5032-2pin_5.0x3.2mm, symbol Device:Crystal
- added C16, C28: 1u, Capacitor_SMD:C_0805_2012Metric, symbol Device:C
- added C20, C22, C23, C25, C26, C32, C33: 100n, Capacitor_SMD:C_0805_2012Metric, symbol Device:C
- added C21, C29, C31: 10u, Capacitor_SMD:C_0805_2012Metric, symbol Device:C
- added CP27: 68u, Capacitor_Tantalum_SMD:CP_EIA-7343-30_AVX-N, symbol Device:CP
- added D1: LED, LED_SMD:LED_1206_3216Metric, symbol Device:LED
- added H1, H2: MountingHole, myFootprints:MountingHole_1.5mm, symbol Mechanical:MountingHole
- added J1: 54548-2271_connector_RPi_zero, myFootprints:545482271_RPi_Zero_connector, symbol myParts:54548-2271_connector_RPi_zero
- added J10, J12, J14, J16: Conn_01x01, TestPoint:TestPoint_Pad_2.0x2.0mm, symbol Connector_Generic:Conn_01x01
- added J11, J13, J15: Conn_01x01, TestPoint:TestPoint_Pad_1.0x1.0mm, symbol Connector_Generic:Conn_01x01
- added J17, J18: Conn_01x01, TestPoint:TestPoint_Pad_4.0x4.0mm, symbol Connector_Generic:Conn_01x01
- added J7: Conn_01x02, Resistor_SMD:R_0603_1608Metric, symbol Connector_Generic:Conn_01x02
- added J9: Conn_01x03, Jumper:SolderJumper-3_P1.3mm_Bridged2Bar12_RoundedPad1.0x1.5mm, symbol Connector_Generic:Conn_01x03
- added U1: LP5907MFX-1.8, Package_TO_SOT_SMD:SOT-23-5, symbol Regulator_Linear:LP5907MFX-1.8
- added U3: LP5907MFX-1.2, Package_TO_SOT_SMD:SOT-23-5, symbol Regulator_Linear:LP5907MFX-1.2
- added U4: LP5907MFX-2.8, Package_TO_SOT_SMD:SOT-23-5, symbol Regulator_Linear:LP5907MFX-2.8
- added U5: PCA9306, Package_SO:SSOP-8_2.95x2.8mm_P0.65mm, symbol Interface:PCA9306
- added U6: TPS82130, Package_LGA:Texas_SIL0008D_MicroSiP-8-1EP_2.8x3mm_P0.65mm_EP1.1x1.9mm_ThermalVias, symbol Regulator_Switching:TPS82130
- added Y1: DSC6011JI1A-008.0000_clock_source, myFootprints:DSC6011JI1A0080000_clock_source, symbol myParts:DSC6011JI1A-008.0000_clock_source
- C1: value 10u -> 1u; footprint Capacitors_SMD:C_0805 -> Capacitor_SMD:C_0805_2012Metric
- C10: value 430p, 1m -> 430p; footprint Capacitors_SMD:C_0805 -> Capacitor_SMD:C_0805_2012Metric
- C11: value 22u -> 100n; footprint Capacitors_SMD:C_0805 -> Capacitor_SMD:C_0805_2012Metric
- C12: value 10u -> 100n; footprint Capacitors_SMD:C_0805 -> Capacitor_SMD:C_0805_2012Metric
- C13: value 100u -> 10u; footprint Capacitors_SMD:C_0805 -> Capacitor_SMD:C_0805_2012Metric
- C14, C3: value 430p, 1m -> 1u; footprint Capacitors_SMD:C_0805 -> Capacitor_SMD:C_0805_2012Metric
- C15: value 100u -> 1u; footprint Capacitors_SMD:C_0805 -> Capacitor_SMD:C_0805_2012Metric
- C17: value 22u -> 1u; footprint Capacitors_SMD:C_0805 -> Capacitor_SMD:C_0805_2012Metric
- C18, C19, C2, C4, C5, C6, C7: footprint Capacitors_SMD:C_0805 -> Capacitor_SMD:C_0805_2012Metric
- C8: value 22u -> 10u; footprint Capacitors_SMD:C_0805 -> Capacitor_SMD:C_0805_2012Metric
- C9: value 10u, 2.229 mOhm -> 10u; footprint Capacitors_SMD:C_0805 -> Capacitor_SMD:C_0805_2012Metric
- J2: footprint Pin_Headers:Pin_Header_Straight_1x01_Pitch2.54mm -> Connector_PinHeader_2.54mm:PinHeader_1x01_P2.54mm_Vertical
- J3: footprint Pin_Headers:Pin_Header_Straight_1x04_Pitch2.54mm -> Connector_PinHeader_2.54mm:PinHeader_1x04_P2.54mm_Vertical
- J4: footprint Pin_Headers:Pin_Header_Straight_1x01_Pitch2.54mm -> TestPoint:TestPoint_Pad_D1.5mm
- J5, J6: footprint Pin_Headers:Pin_Header_Straight_1x04_Pitch2.54mm -> Connector_PinHeader_2.54mm:PinHeader_2x02_P2.54mm_Vertical
- L1: footprint Inductors:Inductor_1212 -> Inductor_SMD:L_1210_3225Metric
- MK1, MK2, MK3, MK4: footprint Mounting_Holes:MountingHole_2.7mm -> MountingHole:MountingHole_3.2mm_M3
- R1, R2: value 10k -> 1k5; footprint Resistors_SMD:R_0805 -> Resistor_SMD:R_0805_2012Metric
- R17, R6, R7: footprint Resistors_SMD:R_0805 -> Resistor_SMD:R_0805_2012Metric
- R3: value 100k -> 200k; footprint Resistors_SMD:R_0805 -> Resistor_SMD:R_0805_2012Metric
- SW1: footprint Buttons_Switches_SMD:SW_SPST_EVPBF -> Button_Switch_SMD:SW_SPST_EVPBF
- U2: footprint myFootprints:MLX75027 -> myFootprints:MLX75027_NSMD
Connections:
- net +12V: now also CP27.1, U6.1 (EN), U6.2 (VIN); no longer C1.1, C12.1, C18.1, C19.1
- net +1V2: now also R7.2, C29.1, C31.1, C32.1, C33.1, J16.1 (Pin_1), U6.4 (VOUT), U6.5 (VOUT); no longer C13.1, C15.1
- net +1V8: now also C11.1, C12.1, C3.1, C8.1, C25.2, C28.2, J10.1 (Pin_1), J9.3 (Pin_3), U1.5 (OUT), U5.2 (VREF1), Y1.1 (OE/STBY/FS), Y1.4 (VDD); no longer C17.1
- net 3V3_Pi: now also C1.1, C13.1, C14.1, C15.1, R3.2, D1.2 (A), J1.22, U1.1 (IN), U1.3 (EN), U3.1 (IN), U3.3 (EN), U4.1 (IN), U4.3 (EN)
- net CLK+: now also J1.9
- net CLK-: now also J1.8
- net D1+: now also J1.3
- net D1-: now also J1.2
- net D2+: now also J1.6
- net D2-: now also J1.5
- net D3+: now also J1.12
- net D3-: now also J1.11
- net D4+: now also J1.15
- net D4-: now also J1.14
- net GNDA: now also C17.2, C19.2, L1.2, C21.2, C23.2, C26.2, U4.2 (GND); no longer C1.2, C3.2, C8.2, L1.1, R3.1
- net GNDD: now also C1.2, C3.2, C8.2, L1.1, MK1.1, MK2.1, MK3.1, MK4.1, C16.2, C20.2, C22.2, C25.1, C28.1, C29.2, C31.2, C32.2, C33.2, CP27.2, D1.1 (K), J1.1, J1.10, J1.13, J1.16, J1.19, J1.23, J1.24, J1.4, J1.7, J17.1 (Pin_1), J18.1 (Pin_1), J9.1 (Pin_1), U1.2 (GND), U3.2 (GND), U5.1 (GND), U6.3 (GND), U6.9 (GND), Y1.2 (GND); no longer C17.2, C19.2, L1.2
- net SCL_Pi: now also J1.20, U5.6 (SCL2)
- net SDA_Pi: now also J1.21, U5.5 (SDA2)
- net VDD: now also C18.1, C16.1, C20.1, J11.1 (Pin_1), U3.5 (OUT); no longer C11.1, R7.2
- net VDDA: now also C17.1, C19.1, C21.1, C23.1, C26.1, J13.1 (Pin_1), U4.5 (OUT); no longer C8.1
- net at U2.A4 (SLASEL): now also J9.2 (Pin_2)
- net SCL: now reaches R1.2
- net SCL: now also U2.B5 (SCL), J12.1 (Pin_1), U5.3 (SCL1); no longer U2.A5 (SDA)
- net CLK: now reaches U2.B3 (CLK)
- net CLK: now also J15.1 (Pin_1), Y1.3 (OUT)
- net SDA: now reaches R2.2
- net SDA: now also U2.A5 (SDA), J14.1 (Pin_1), U5.4 (SDA1); no longer U2.B5 (SCL)
- net at R6.2, R7.1: now also U6.6 (FB)
- net at C10.1: now also U6.8 (SS/TR)
- new net: J1.18, J7.1 (Pin_1)
- new net: J1.17, J7.2 (Pin_2)
- new net: C22.1, R3.1, U5.7 (VREF2), U5.8 (EN)
- no-connect marks 6 -> 1
Other:
- note added: "Clock generator: \nDSC6011JI1A-008.0000"
- note added: "It is completely fucked up. 22 pin connector is inverted on camera side. My mistake was interpreting it as the one on RPi Zero :-("
- note added: "LED: 156120GS75300"
- note added: "NO BARREL JACK\n\nMODEL: PJ-002AH"
- note added: "System voltages:\nVDDA - 2.7 V, 40 mA\n TI 2.8 VLDO\nVDDMIX - 1.2 V, 3 A\n TI TPS82130\nVDDD - 1.2 V, 200 mA\n TI LDO\nVDDIF - 1.8 V, 3 mA\n TI LDO"
- note added: "TPSE686K020R0150"
- note removed: "+3.3v -1\nSDA - 2\nSCL - 3"
- note removed: "15 - +3.3 V\n14 - SDA \n13 - SCL\n12 - GPIO1\n11 - GPIO0\n10 - GND\n9 - CLK+\n8 - CLK-\n7 - GND\n6 - D1+\n5 - D1-\n4 - GND\n3 - D0+\n2 - D0-\n1 - GND"
- note removed: "C3, C10 and C14\n 430pF or 3.3nF???\n"
- note removed: "GND - 13\nCLK+ - 14\nCLK- - 15\nGND - 16\nD1+ - 17\nD1- - 18\nGND - 19\nD0+ - 20\nD0- - 21\nGND - 22"
- note removed: "GND - 7\nD3+ - 8\nD3- - 9\nGND - 10\nD2+ - 11\nD2- - 12"
- note removed: "GPIO1 -5\nGPIO0 -6"
- note removed: "It isn't exact drawing, but connectors should be connected in similar way using standard Raspberry Pi cable-adapter"
- note removed: "J3 connector on Zynqberry is rotated, so that our connector can be drawn in regular manner"
- note removed: "System voltages:\nVDDA - 2.7 V, 0.2 A\n TI TPS82150\nVDDMIX - 1.2 V, 6 A\n TI tpsm84824\nVDDD - 1.2 V, 0.5 A\n TI TPS82150\nVDDIF - 1.8 V, 0.05 A\n TI TPS82150"
- note removed: "nc - 4"
- moved on the sheet: C10, C2, C4, C5, C6, C7, C9, J2, J3, J4, J5, J6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
